File: PrototypeNumpad.kicad_pcb (KiCad board)
At the start: 2 copper layers, 99 x 99 mm, 86 parts, among them J0 Conn_01x06, J1 USB_B_Micro, SW0 SW_Push, U1 ATmega32U4-AU, U2 USBLC6-2SC6, Y1 Crystal_GND24

Commit message: Route tracks
Parts:
- moved C7 27.9 mm to (79.8, 63.5), turned to 90 degrees
- moved C3 19.8 mm to (78.5, 73.0)
- moved C6 14.7 mm to (97.5, 73.2), turned to 90 degrees
- moved C5 11.7 mm to (99.3, 65.8)
- moved C10 11.4 mm to (103.5, 49.5)
- moved C8 3.42 mm to (76.8, 63.5), turned to 90 degrees
- moved Y1 0.90 mm to (84.8, 49.5), turned to 270 degrees
Routing:
- net VCC: track 0.00 -> 449.1 mm, vias 0 -> 10
- net RowE: track 0.00 -> 143.3 mm, vias 0 -> 2
- net Col5: track 0.00 -> 132.4 mm, vias 0 -> 1
- net RowD: track 0.00 -> 117.9 mm, vias 0 -> 2
- net Col3: track 0.00 -> 115.1 mm, vias 0 -> 3
- net Col1: track 0.00 -> 107.8 mm, vias 0 -> 1
- net RowC: track 0.00 -> 102.8 mm, vias 0 -> 2
- net Col4: track 0.00 -> 102.6 mm
- net RowA: track 0.00 -> 93.7 mm
- net RowB: track 0.00 -> 92.3 mm, vias 0 -> 5
- net Col2: track 0.00 -> 84.1 mm, vias 0 -> 1
- net GND: track 0.00 -> 78.0 mm, vias 0 -> 20
- net Net-(D4-Pad2): track 0.00 -> 68.0 mm
- net RST: track 0.00 -> 67.1 mm, vias 0 -> 3
- net Net-(D3-Pad2): track 0.00 -> 58.8 mm
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