File: PrototypeNumpad.sch (KiCad schematic (older format))
At the start: 65 parts, among them J1 USB_B_Micro, SW0 SW_Push, U1 ATmega32U4-AU, Y1 Crystal_GND3

Commit message: Add ISP connectors
Parts:
- added J0: Conn_01x06, symbol Connector_Generic:Conn_01x06
Connections:
- net labels added: MISO, MOSI, RST, SCK
- wire segments 120 -> 124

Commit message: Add RGB underglow
Parts:
- added C10, C11, C12, C13, C14, C15: 0.1uF, symbol Device:C
- added C9: 47uF, symbol Device:C
- added D1, D2, D3, D4, D5, D6: WS2812B, LED_SMD:LED_WS2812B_PLCC4_5.0x5.0mm_P3.2mm, symbol LED:WS2812B
- added R5: 470, symbol Device:R
Connections:
- net labels added: RGB
- wire segments 124 -> 163

Commit message: Add switch A1
Parts:
- added D_A1: D, symbol Device:D
- added SW_A1: SW_Push, symbol Switch:SW_Push
- gave numbers to parts that had none: 1
Connections:
- wire segments 163 -> 165
Changed lines of the file:
@@
 $EndComp
 $Comp
-L power:GND #PWR?
+L power:GND #PWR0101
 U 1 1 5BB1ABFB
 P 4250 7250
-F 0 "#PWR?" H 4250 7000 50  0001 C CNN
+F 0 "#PWR0101" H 4250 7000 50  0001 C CNN
 F 1 "GND" H 4255 7077 50  0000 C CNN
 F 2 "" H 4250 7250 50  0001 C CNN
@@
 	4400 6750 4550 6750
 $Comp
-L power:VCC #PWR?
+L power:VCC #PWR0102
 U 1 1 5BB1B7F7
 P 3600 5500
-F 0 "#PWR?" H 3600 5350 50  0001 C CNN
+F 0 "#PWR0102" H 3600 5350 50  0001 C CNN
 F 1 "VCC" H 3617 5673 50  0000 C CNN
 F 2 "" H 3600 5500 50  0001 C CNN
@@
 	3600 5500 3600 5600
 $Comp
-L power:GND #PWR?
+L power:GND #PWR0103
 U 1 1 5BB1CF48
 P 3600 6150
-F 0 "#PWR?" H 3600 5900 50  0001 C CNN
+F 0 "#PWR0103" H 3600 5900 50  0001 C CNN
 F 1 "GND" H 3605 5977 50  0000 C CNN
 F 2 "" H 3600 6150 50  0001 C CNN
@@
 	3050 5900 3200 5900
 $Comp
-L power:GND #PWR?
+L power:GND #PWR0104
 U 1 1 5BB483FD
 P 1000 6300
-F 0 "#PWR?" H 1000 6050 50  0001 C CNN
+F 0 "#PWR0104" H 1000 6050 50  0001 C CNN
 F 1 "GND" H 1005 6127 50  0000 C CNN
 F 2 "" H 1000 6300 50  0001 C CNN
@@
 $EndComp
 $Comp
-L power:GND #PWR?
+L power:GND #PWR0105
 U 1 1 5BB48D61
 P 2050 7250
-F 0 "#PWR?" H 2050 7000 50  0001 C CNN
+F 0 "#PWR0105" H 2050 7000 50  0001 C CNN
 F 1 "GND" H 2055 7077 50  0000 C CNN
 F 2 "" H 2050 7250 50  0001 C CNN
@@
 $EndComp
 $Comp
-L Power_Protection:USBLC6-2SC6 U?
+L Power_Protection:USBLC6-2SC6 U2
 U 1 1 5BB20C4F
 P 2050 6750
-F 0 "U?" H 2050 7428 50  0000 C CNN
+F 0 "U2" H 2050 7428 50  0000 C CNN
 F 1 "USBLC6-2SC6" H 2050 7337 50  0000 C CNN
 F 2 "Package_TO_SOT_SMD:SOT-23-6" H 1300 7150 50  0001 C CNN
@@
 $EndComp
 $Comp
-L power:VCC #PWR?
+L power:VCC #PWR0106
 U 1 1 5BB4983C
 P 3200 5500
-F 0 "#PWR?" H 3200 5350 50  0001 C CNN
+F 0 "#PWR0106" H 3200 5350 50  0001 C CNN
 F 1 "VCC" H 3217 5673 50  0000 C CNN
 F 2 "" H 3200 5500 50  0001 C CNN
@@
 	1550 2550 1350 2550
 $Comp
-L power:GND #PWR?
+L power:GND #PWR0107
 U 1 1 5BB525A9
 P 1350 3200
-F 0 "#PWR?" H 1350 2950 50  0001 C CNN
+F 0 "#PWR0107" H 1350 2950 50  0001 C CNN
 F 1 "GND" H 1355 3027 50  0000 C CNN
 F 2 "" H 1350 3200 50  0001 C CNN
@@
 	3200 5600 3200 5500
 $Comp
-L power:VCC #PWR?
+L power:VCC #PWR0108
 U 1 1 5BB59BD5
 P 1350 2200
-F 0 "#PWR?" H 1350 2050 50  0001 C CNN
+F 0 "#PWR0108" H 1350 2050 50  0001 C CNN
 F 1 "VCC" H 1367 2373 50  0000 C CNN
 F 2 "" H 1350 2200 50  0001 C CNN
@@
 Connection ~ 2150 1050
 $Comp
-L power:VCC #PWR?
+L power:VCC #PWR0109
 U 1 1 5BB5DDEA
 P 2150 900
-F 0 "#PWR?" H 2150 750 50  0001 C CNN
+F 0 "#PWR0109" H 2150 750 50  0001 C CNN
 F 1 "VCC" H 2167 1073 50  0000 C CNN
 F 2 "" H 2150 900 50  0001 C CNN
@@
 $EndComp
 $Comp
-L power:VCC #PWR?
+L power:VCC #PWR0110
 U 1 1 5BB66D84
 P 1500 900
-F 0 "#PWR?" H 1500 750 50  0001 C CNN
+F 0 "#PWR0110" H 1500 750 50  0001 C CNN
 F 1 "VCC" H 1517 1073 50  0000 C CNN
 F 2 "" H 1500 900 50  0001 C CNN
@@
 	850  1500 850  1450
 $Comp
-L power:GND #PWR?
+L power:GND #PWR0111
 U 1 1 5BB6381D
 P 850 1500
-F 0 "#PWR?" H 850 1250 50  0001 C CNN
+F 0 "#PWR0111" H 850 1250 50  0001 C CNN
 F 1 "GND" H 855 1327 50  0000 C CNN
 F 2 "" H 850 1500 50  0001 C CNN
@@
 	850  1450 950  1450
 $Comp
-L power:GND #PWR?
+L power:GND #PWR0112
 U 1 1 5BB937E8
 P 3150 3650
-F 0 "#PWR?" H 3150 3400 50  0001 C CNN
+F 0 "#PWR0112" H 3150 3400 50  0001 C CNN
 F 1 "GND" H 3155 3477 50  0000 C CNN
 F 2 "" H 3150 3650 50  0001 C CNN
@@
 	1000 6250 1000 6200
 $Comp
-L power:GND #PWR?
+L power:GND #PWR0113
 U 1 1 5BBD54B8
 P 2150 4850
-F 0 "#PWR?" H 2150 4600 50  0001 C CNN
+F 0 "#PWR0113" H 2150 4600 50  0001 C CNN
 F 1 "GND" H 2155 4677 50  0000 C CNN
 F 2 "" H 2150 4850 50  0001 C CNN
@@
 Connection ~ 2150 4800
 Wire Wire Line
-	3600 1100 3600 2250
-$Comp
-L power:GND #PWR?
+	3600 1100 3600 1550
+$Comp
+L power:GND #PWR0114
 U 1 1 5BBEFC9F
 P 5500 5950
-F 0 "#PWR?" H 5500 5700 50  0001 C CNN
+F 0 "#PWR0114" H 5500 5700 50  0001 C CNN
 F 1 "GND" H 5505 5777 50  0000 C CNN
 F 2 "" H 5500 5950 50  0001 C CNN
@@
 MISO
 $Comp
-L power:VCC #PWR?
+L power:VCC #PWR0115
 U 1 1 5BC20F33
 P 5900 5950
-F 0 "#PWR?" H 5900 5800 50  0001 C CNN
+F 0 "#PWR0115" H 5900 5800 50  0001 C CNN
 F 1 "VCC" H 5917 6123 50  0000 C CNN
 F 2 "" H 5900 5950 50  0001 C CNN
@@
 $EndComp
 $Comp
-L power:VCC #PWR?
+L power:VCC #PWR0116
 U 1 1 5BD40317
 P 8000 1250
-F 0 "#PWR?" H 8000 1100 50  0001 C CNN
+F 0 "#PWR0116" H 8000 1100 50  0001 C CNN
 F 1 "VCC" H 8017 1423 50  0000 C CNN
 F 2 "" H 8000 1250 50  0001 C CNN
@@
 $EndComp
 $Comp
-L power:GND #PWR?
+L power:GND #PWR0117
 U 1 1 5BD404D8
 P 8000 1850
-F 0 "#PWR?" H 8000 1600 50  0001 C CNN
+F 0 "#PWR0117" H 8000 1600 50  0001 C CNN
 F 1 "GND" H 8005 1677 50  0000 C CNN
 F 2 "" H 8000 1850 50  0001 C CNN
@@
 $EndComp
 $Comp
-L power:VCC #PWR?
+L power:VCC #PWR0118
 U 1 1 5BD40708
 P 8750 1250
-F 0 "#PWR?" H 8750 1100 50  0001 C CNN
+F 0 "#PWR0118" H 8750 1100 50  0001 C CNN
 F 1 "VCC" H 8767 1423 50  0000 C CNN
 F 2 "" H 8750 1250 50  0001 C CNN
@@
 $EndComp
 $Comp
-L power:GND #PWR?
+L power:GND #PWR0119
 U 1 1 5BD4070E
 P 8750 1850
-F 0 "#PWR?" H 8750 1600 50  0001 C CNN
+F 0 "#PWR0119" H 8750 1600 50  0001 C CNN
 F 1 "GND" H 8755 1677 50  0000 C CNN
 F 2 "" H 8750 1850 50  0001 C CNN
@@
 $EndComp
 $Comp
-L power:VCC #PWR?
+L power:VCC #PWR0120
 U 1 1 5BD4454A
 P 9500 1250
-F 0 "#PWR?" H 9500 1100 50  0001 C CNN
+F 0 "#PWR0120" H 9500 1100 50  0001 C CNN
 F 1 "VCC" H 9517 1423 50  0000 C CNN
 F 2 "" H 9500 1250 50  0001 C CNN
@@
 $EndComp
 $Comp
-L power:GND #PWR?
+L power:GND #PWR0121
 U 1 1 5BD44550
 P 9500 1850
-F 0 "#PWR?" H 9500 1600 50  0001 C CNN
+F 0 "#PWR0121" H 9500 1600 50  0001 C CNN
 F 1 "GND" H 9505 1677 50  0000 C CNN
 F 2 "" H 9500 1850 50  0001 C CNN
@@
 $EndComp
 $Comp
-L power:VCC #PWR?
+L power:VCC #PWR0122
 U 1 1 5BD485E3
 P 8000 2350
-F 0 "#PWR?" H 8000 2200 50  0001 C CNN
+F 0 "#PWR0122" H 8000 2200 50  0001 C CNN
 F 1 "VCC" H 8017 2523 50  0000 C CNN
 F 2 "" H 8000 2350 50  0001 C CNN
@@
 $EndComp
 $Comp
-L power:GND #PWR?
+L power:GND #PWR0123
 U 1 1 5BD485E9
 P 8000 2950
-F 0 "#PWR?" H 8000 2700 50  0001 C CNN
+F 0 "#PWR0123" H 8000 2700 50  0001 C CNN
 F 1 "GND" H 8005 2777 50  0000 C CNN
 F 2 "" H 8000 2950 50  0001 C CNN
@@
 $EndComp
 $Comp
-L power:VCC #PWR?
+L power:VCC #PWR0124
 U 1 1 5BD4C557
 P 8750 2350
-F 0 "#PWR?" H 8750 2200 50  0001 C CNN
+F 0 "#PWR0124" H 8750 2200 50  0001 C CNN
 F 1 "VCC" H 8767 2523 50  0000 C CNN
 F 2 "" H 8750 2350 50  0001 C CNN
@@
 $EndComp
 $Comp
-L power:GND #PWR?
+L power:GND #PWR0125
 U 1 1 5BD4C55D
 P 8750 2950
-F 0 "#PWR?" H 8750 2700 50  0001 C CNN
+F 0 "#PWR0125" H 8750 2700 50  0001 C CNN
 F 1 "GND" H 8755 2777 50  0000 C CNN
 F 2 "" H 8750 2950 50  0001 C CNN
@@
 $EndComp
 $Comp
-L power:VCC #PWR?
+L power:VCC #PWR0126
 U 1 1 5BD503A4
 P 9500 2350
-F 0 "#PWR?" H 9500 2200 50  0001 C CNN
+F 0 "#PWR0126" H 9500 2200 50  0001 C CNN
 F 1 "VCC" H 9517 2523 50  0000 C CNN
 F 2 "" H 9500 2350 50  0001 C CNN
@@
 $EndComp
 $Comp
-L power:GND #PWR?
+L power:GND #PWR0127
 U 1 1 5BD503AA
 P 9500 2950
-F 0 "#PWR?" H 9500 2700 50  0001 C CNN
+F 0 "#PWR0127" H 9500 2700 50  0001 C CNN
 F 1 "GND" H 9505 2777 50  0000 C CNN
 F 2 "" H 9500 2950 50  0001 C CNN
@@
 	7350 1550 7300 1550
 $Comp
-L power:VCC #PWR?
+L power:VCC #PWR0128
 U 1 1 5BDC1CBB
 P 7650 3450
-F 0 "#PWR?" H 7650 3300 50  0001 C CNN
+F 0 "#PWR0128" H 7650 3300 50  0001 C CNN
 F 1 "VCC" H 7667 3623 50  0000 C CNN
 F 2 "" H 7650 3450 50  0001 C CNN
@@
 Connection ~ 7650 3950
 $Comp
-L power:GND #PWR?
+L power:GND #PWR0129
 U 1 1 5BDCCE62
 P 7650 4100
-F 0 "#PWR?" H 7650 3850 50  0001 C CNN
+F 0 "#PWR0129" H 7650 3850 50  0001 C CNN
 F 1 "GND" H 7655 3927 50  0000 C CNN
 F 2 "" H 7650 4100 50  0001 C CNN
@@
 Wire Wire Line
 	9400 3550 9750 3550
+$Comp
+L Switch:SW_Push SW_A1
+U 1 1 5BBDBE6D
+P 3800 1550
+F 0 "SW_A1" H 3800 1835 50  0000 C CNN
+F 1 "SW_Push" H 3800 1744 50  0000 C CNN
+F 2 "" H 3800 1750 50  0001 C CNN
+F 3 "" H 3800 1750 50  0001 C CNN
+	1    3800 1550
+	1    0    0    -1
+$EndComp
+Connection ~ 3600 1550
+Wire Wire Line
+	3600 1550 3600 2250
+$Comp
+L Device:D D_A1
+U 1 1 5BBDBF29
+P 4000 1700
+F 0 "D_A1" V 4046 1621 50  0000 R CNN
+F 1 "D" V 3955 1621 50  0000 R CNN
+F 2 "" H 4000 1700 50  0001 C CNN
+F 3 "~" H 4000 1700 50  0001 C CNN
+	1    4000 1700
+	0    1    -1   0
+$EndComp
+Wire Wire Line
+	4000 1850 4600 1850
+Connection ~ 4600 1850
 $EndSCHEMATC

Commit message: Assign PCB footprints to schematic symbols
Parts:
- C1, C10, C11, C12, C13, C14, C15, C2, C3, C4, C5, C6, C7, C8: footprint (none) -> Capacitor_SMD:C_1206_3216Metric_Pad1.42x1.75mm_HandSolder
- C9: footprint (none) -> Capacitor_SMD:C_0805_2012Metric_Pad1.15x1.40mm_HandSolder
- D_A1, D_A2, D_A3, D_A4, D_A5, D_B1, D_B2, D_B3, D_B4, D_B5, D_C1, D_C2, D_C3, D_C4, D_C5, D_D1, D_D2, D_D3, D_D4, D_D5, D_E1, D_E2, D_E3, D_E4, D_E5: footprint (none) -> Diode_SMD:D_SOD-123
- J0: footprint (none) -> Connector_PinHeader_2.54mm:PinHeader_1x06_P2.54mm_Vertical
- J1: footprint (none) -> Connector_USB:USB_Micro-B_Molex-105017-0001
- R1, R2, R3, R4, R5: footprint (none) -> Resistor_SMD:R_1206_3216Metric_Pad1.42x1.75mm_HandSolder
- SW0: footprint (none) -> Button_Switch_SMD:SW_SPST_TL3342
- SW_A1, SW_A2, SW_A3, SW_A4, SW_A5, SW_B1, SW_B2, SW_B3, SW_B4, SW_B5, SW_C1, SW_C2, SW_C3, SW_C4, SW_C5, SW_D1, SW_D2, SW_D3, SW_D4, SW_D5, SW_E1, SW_E2, SW_E3, SW_E4, SW_E5: footprint (none) -> Button_Switch_Keyboard:SW_Cherry_MX1A_1.00u_PCB
- Y1: footprint (none) -> Crystal:Crystal_SMD_SeikoEpson_FA238-4Pin_3.2x2.5mm_HandSoldering

Commit message: Change Crystal grounding pins
Parts:
- removed Y1: Crystal_GND3, Crystal:Crystal_SMD_SeikoEpson_FA238-4Pin_3.2x2.5mm_HandSoldering, symbol Device:Crystal_GND3
- added Y1: Crystal_GND24, Crystal:Crystal_SMD_SeikoEpson_FA238-4Pin_3.2x2.5mm_HandSoldering, symbol Device:Crystal_GND24
Connections:
- wire segments 165 -> 170
Changed lines of the file:
@@
-$EndComp
-$Comp
-L Device:Crystal_GND3 Y1
-U 1 1 5BB1A802
-P 4250 6750
-F 0 "Y1" H 4250 7018 50  0000 C CNN
-F 1 "Crystal_GND3" H 4250 6927 50  0000 C CNN
-F 2 "Crystal:Crystal_SMD_SeikoEpson_FA238-4Pin_3.2x2.5mm_HandSoldering" H 4250 6750 50  0001 C CNN
-F 3 "~" H 4250 6750 50  0001 C CNN
-	1    4250 6750
-	1    0    0    -1
 $EndComp
 $Comp
@@
 	3950 7050 4250 7050
 Wire Wire Line
-	4250 7050 4250 7250
+	4250 7050 4250 7150
 Connection ~ 4250 7050
 Wire Wire Line
@@
 	4000 1850 4600 1850
 Connection ~ 4600 1850
+$Comp
+L Device:Crystal_GND24 Y1
+U 1 1 5BBF5CB1
+P 4250 6750
+F 0 "Y1" H 4200 7100 50  0000 L CNN
+F 1 "Crystal_GND24" H 4000 7000 50  0000 L CNN
+F 2 "Crystal:Crystal_SMD_SeikoEpson_FA238-4Pin_3.2x2.5mm_HandSoldering" H 4250 6750 50  0001 C CNN
+F 3 "~" H 4250 6750 50  0001 C CNN
+	1    4250 6750
+	1    0    0    -1
+$EndComp
+Wire Wire Line
+	3600 7150 4250 7150
+Connection ~ 4250 7150
+Wire Wire Line
+	4250 7150 4250 7250
+Wire Wire Line
+	4250 6550 4250 6500
+Wire Wire Line
+	4250 6500 3600 6500
+Wire Wire Line
+	3600 6500 3600 7150
 $EndSCHEMATC

Commit message: Add M2.5 mounting holes
Parts:
- added MH0, MH1, MH2, MH3: MountingHole, MountingHole:MountingHole_2.5mm_Pad, symbol Mechanical:MountingHole
Changed lines of the file:
@@
 Wire Wire Line
 	3600 6500 3600 7150
+$Comp
+L Mechanical:MountingHole MH0
+U 1 1 5BC3C1C0
+P 5500 6600
+F 0 "MH0" H 5600 6646 50  0000 L CNN
+F 1 "MountingHole" H 5600 6555 50  0000 L CNN
+F 2 "MountingHole:MountingHole_2.5mm_Pad" H 5500 6600 50  0001 C CNN
+F 3 "~" H 5500 6600 50  0001 C CNN
+	1    5500 6600
+	1    0    0    -1
+$EndComp
+$Comp
+L Mechanical:MountingHole MH1
+U 1 1 5BC3CC1B
+P 5500 6800
+F 0 "MH1" H 5600 6846 50  0000 L CNN
+F 1 "MountingHole" H 5600 6755 50  0000 L CNN
+F 2 "MountingHole:MountingHole_2.5mm_Pad" H 5500 6800 50  0001 C CNN
+F 3 "~" H 5500 6800 50  0001 C CNN
+	1    5500 6800
+	1    0    0    -1
+$EndComp
+$Comp
+L Mechanical:MountingHole MH2
+U 1 1 5BC3CCDF
+P 5500 7000
+F 0 "MH2" H 5600 7046 50  0000 L CNN
+F 1 "MountingHole" H 5600 6955 50  0000 L CNN
+F 2 "MountingHole:MountingHole_2.5mm_Pad" H 5500 7000 50  0001 C CNN
+F 3 "~" H 5500 7000 50  0001 C CNN
+	1    5500 7000
+	1    0    0    -1
+$EndComp
+$Comp
+L Mechanical:MountingHole MH3
+U 1 1 5BC3CD9D
+P 5500 7200
+F 0 "MH3" H 5600 7246 50  0000 L CNN
+F 1 "MountingHole" H 5600 7155 50  0000 L CNN
+F 2 "MountingHole:MountingHole_2.5mm_Pad" H 5500 7200 50  0001 C CNN
+F 3 "~" H 5500 7200 50  0001 C CNN
+	1    5500 7200
+	1    0    0    -1
+$EndComp
 $EndSCHEMATC

Commit message: Expose USB traces as headers
Parts:
- added J1A1: Conn_01x04, Connector_PinHeader_2.54mm:PinHeader_1x04_P2.54mm_Vertical, symbol Connector_Generic:Conn_01x04
Connections:
- wire segments 170 -> 172
Changed lines of the file:
@@
 	1    0    0    -1
 $EndComp
+$Comp
+L Connector_Generic:Conn_01x04 J1A1
+U 1 1 5BC0A72D
+P 6750 5600
+F 0 "J1A1" V 6716 5312 50  0000 R CNN
+F 1 "Conn_01x04" V 6625 5312 50  0000 R CNN
+F 2 "Connector_PinHeader_2.54mm:PinHeader_1x04_P2.54mm_Vertical" H 6750 5600 50  0001 C CNN
+F 3 "~" H 6750 5600 50  0001 C CNN
+	1    6750 5600
+	0    -1   -1   0
+$EndComp
+Text GLabel 6750 5800 3    50   Input ~ 0
+D+
+Text GLabel 6850 5800 3    50   Input ~ 0
+D-
+$Comp
+L power:VCC #PWR0130
+U 1 1 5BC12FE9
+P 6950 5950
+F 0 "#PWR0130" H 6950 5800 50  0001 C CNN
+F 1 "VCC" H 6967 6123 50  0000 C CNN
+F 2 "" H 6950 5950 50  0001 C CNN
+F 3 "" H 6950 5950 50  0001 C CNN
+	1    6950 5950
+	-1   0    0    1
+$EndComp
+$Comp
+L power:GND #PWR0131
+U 1 1 5BC1381C
+P 6650 5950
+F 0 "#PWR0131" H 6650 5700 50  0001 C CNN
+F 1 "GND" H 6655 5777 50  0000 C CNN
+F 2 "" H 6650 5950 50  0001 C CNN
+F 3 "" H 6650 5950 50  0001 C CNN
+	1    6650 5950
+	1    0    0    -1
+$EndComp
+Wire Wire Line
+	6650 5950 6650 5800
+Wire Wire Line
+	6950 5950 6950 5800
 $EndSCHEMATC

Commit message: Add Speaker
Parts:
- added BZ1: Buzzer, Fate_Parts:Buzzer_AST1109MLTRQ, symbol Device:Buzzer
- added C16: 10uF, Capacitor_SMD:C_1206_3216Metric_Pad1.42x1.75mm_HandSolder, symbol Device:C
- added Q1: 2N7002, Package_TO_SOT_SMD:SOT-23_Handsoldering, symbol Transistor_FET:2N7002
- added R6: 470, Resistor_SMD:R_1206_3216Metric_Pad1.42x1.75mm_HandSolder, symbol Device:R
- added R7: 10K, Resistor_SMD:R_1206_3216Metric_Pad1.42x1.75mm_HandSolder, symbol Device:R
Connections:
- net labels added: SPEAKER
- wire segments 172 -> 174
Changed lines of the file:
@@
 Wire Wire Line
 	6950 5950 6950 5800
+$Comp
+L Transistor_FET:2N7002 Q1
+U 1 1 5BC67172
+P 8200 5650
+F 0 "Q1" H 8405 5696 50  0000 L CNN
+F 1 "2N7002" H 8405 5605 50  0000 L CNN
+F 2 "Package_TO_SOT_SMD:SOT-23_Handsoldering" H 8400 5575 50  0001 L CIN
+F 3 "https://www.fairchildsemi.com/datasheets/2N/2N7002.pdf" H 8200 5650 50  0001 L CNN
+	1    8200 5650
+	1    0    0    -1
+$EndComp
+Text GLabel 8000 5650 0    50   Input ~ 0
+SPEAKER
+Text GLabel 2750 2350 2    50   Input ~ 0
+SPEAKER
+$Comp
+L power:GND #PWR0132
+U 1 1 5BCAFA46
+P 8000 5950
+F 0 "#PWR0132" H 8000 5700 50  0001 C CNN
+F 1 "GND" H 8005 5777 50  0000 C CNN
+F 2 "" H 8000 5950 50  0001 C CNN
+F 3 "" H 8000 5950 50  0001 C CNN
+	1    8000 5950
+	1    0    0    -1
+$EndComp
+$Comp
+L power:GND #PWR0133
+U 1 1 5BCAFC0E
+P 8300 5850
+F 0 "#PWR0133" H 8300 5600 50  0001 C CNN
+F 1 "GND" H 8305 5677 50  0000 C CNN
+F 2 "" H 8300 5850 50  0001 C CNN
+F 3 "" H 8300 5850 50  0001 C CNN
+	1    8300 5850
+	1    0    0    -1
+$EndComp
+$Comp
+L Device:R R7
+U 1 1 5BCAF104
+P 8000 5800
+F 0 "R7" V 7900 5800 50  0000 C CNN
+F 1 "10K" V 8000 5800 50  0000 C CNN
+F 2 "Resistor_SMD:R_1206_3216Metric_Pad1.42x1.75mm_HandSolder" V 7930 5800 50  0001 C CNN
+F 3 "~" H 8000 5800 50  0001 C CNN
+	1    8000 5800
+	1    0    0    -1
+$EndComp
+$Comp
+L Device:Buzzer BZ1
+U 1 1 5BCCDA13
+P 8200 5350
+F 0 "BZ1" H 8400 5400 50  0000 C CNN
+F 1 "Buzzer" H 8450 5300 50  0000 C CNN
+F 2 "Fate_Parts:Buzzer_AST1109MLTRQ" V 8175 5450 50  0001 C CNN
+F 3 "~" V 8175 5450 50  0001 C CNN
+	1    8200 5350
+	-1   0    0    -1
+$EndComp
+$Comp
+L power:VCC #PWR0134
+U 1 1 5BCCE239
+P 8300 4950
+F 0 "#PWR0134" H 8300 4800 50  0001 C CNN
+F 1 "VCC" H 8317 5123 50  0000 C CNN
+F 2 "" H 8300 4950 50  0001 C CNN
+F 3 "" H 8300 4950 50  0001 C CNN
+	1    8300 4950
+	1    0    0    -1
+$EndComp
+$Comp
+L Device:R R6
+U 1 1 5BCCE8F2
+P 8300 5100
+F 0 "R6" V 8200 5100 50  0000 C CNN
+F 1 "470" V 8300 5100 50  0000 C CNN
+F 2 "Resistor_SMD:R_1206_3216Metric_Pad1.42x1.75mm_HandSolder" V 8230 5100 50  0001 C CNN
+F 3 "~" H 8300 5100 50  0001 C CNN
+	1    8300 5100
+	-1   0    0    1
+$EndComp
+$Comp
+L Device:C C16
+U 1 1 5BCD6A4A
+P 8800 5700
+F 0 "C16" H 8850 5800 50  0000 L CNN
+F 1 "10uF" H 8850 5600 50  0000 L CNN
+F 2 "Capacitor_SMD:C_1206_3216Metric_Pad1.42x1.75mm_HandSolder" H 8838 5550 50  0001 C CNN
+F 3 "~" H 8800 5700 50  0001 C CNN
+	1    8800 5700
+	1    0    0    -1
+$EndComp
+$Comp
+L power:GND #PWR0135
+U 1 1 5BCF2CD8
+P 8800 5850
+F 0 "#PWR0135" H 8800 5600 50  0001 C CNN
+F 1 "GND" H 8805 5677 50  0000 C CNN
+F 2 "" H 8800 5850 50  0001 C CNN
+F 3 "" H 8800 5850 50  0001 C CNN
+	1    8800 5850
+	1    0    0    -1
+$EndComp
+Wire Wire Line
+	8800 5550 8800 5250
+Wire Wire Line
+	8800 5250 8300 5250
+Connection ~ 8300 5250
 $EndSCHEMATC
