File: PrototypeNumpad.sch (KiCad schematic (older format))
At the start: 92 parts, among them J0 Conn_01x06, J1 USB_B_Micro, J1A1 Conn_01x04, Q1 2N7002, SW0 SW_Push, U1 ATmega32U4-AU, U2 USBLC6-2SC6, Y1 Crystal_GND24

Commit message: Update ATmega32u4 decoupling capacitor values
Parts:
- C3: value 0.1uF -> 1uF
- C4: value 1F -> 0.1uF
- C5: value 1uF -> 0.1uF
- C6: value 10uF -> 0.1uF
Changed lines of the file:
@@
 P 3600 5800
 F 0 "C3" H 3650 5900 50  0000 L CNN
-F 1 "0.1uF" H 3650 5700 50  0000 L CNN
+F 1 "1uF" H 3650 5700 50  0000 L CNN
 F 2 "Capacitor_SMD:C_1206_3216Metric_Pad1.42x1.75mm_HandSolder" H 3638 5650 50  0001 C CNN
 F 3 "~" H 3600 5800 50  0001 C CNN
@@
 P 3950 5800
 F 0 "C4" H 4000 5900 50  0000 L CNN
-F 1 "1F" H 4000 5700 50  0000 L CNN
+F 1 "0.1uF" H 4000 5700 50  0000 L CNN
 F 2 "Capacitor_SMD:C_1206_3216Metric_Pad1.42x1.75mm_HandSolder" H 3988 5650 50  0001 C CNN
 F 3 "~" H 3950 5800 50  0001 C CNN
@@
 P 4300 5800
 F 0 "C5" H 4350 5900 50  0000 L CNN
-F 1 "1uF" H 4350 5700 50  0000 L CNN
+F 1 "0.1uF" H 4350 5700 50  0000 L CNN
 F 2 "Capacitor_SMD:C_1206_3216Metric_Pad1.42x1.75mm_HandSolder" H 4338 5650 50  0001 C CNN
 F 3 "~" H 4300 5800 50  0001 C CNN
@@
 P 4650 5800
 F 0 "C6" H 4700 5900 50  0000 L CNN
-F 1 "10uF" H 4700 5700 50  0000 L CNN
+F 1 "0.1uF" H 4700 5700 50  0000 L CNN
 F 2 "Capacitor_SMD:C_1206_3216Metric_Pad1.42x1.75mm_HandSolder" H 4688 5650 50  0001 C CNN
 F 3 "~" H 4650 5800 50  0001 C CNN
